File: Hardware/Qwiic_Shield_for_Photon.sch (EAGLE design)
At the start: 21 parts

Commit message: ran checklist, pre design review
Parts:
- added FD1, FD2, FD3, FD4: FIDUCIALUFIDUCIAL, SparkFun-Aesthetics:FIDUCIALUFIDUCIAL
- added LOGO2: REVISION, SparkFun-Aesthetics:REVISION
- J1, J2, J3: device SparkX:I2C_STANDARDJS-1MM -> SparkFun-Connectors:QWIIC_CONNECTORJS-1MM
- U$4: value SPARKX-LOGO5 -> SFE_LOGO_NAME.1_INCH; device SparkX:SPARKX-LOGO5 -> SparkFun-Aesthetics:SFE_LOGO_NAME.1_INCH
Other:
- note added: "Andy England"
- note added: "v01"
Changed lines of the file:
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@@
 <?xml version="1.0" encoding="utf-8"?>
 <!DOCTYPE eagle SYSTEM "eagle.dtd">
-<eagle version="7.6.0">
+<eagle version="7.7.0">
 <drawing>
 <settings>
@@
 <layer number="230" name="230bmp" color="7" fill="1" visible="yes" active="yes"/>
 <layer number="231" name="231bmp" color="7" fill="1" visible="yes" active="yes"/>
+<layer number="232" name="Eagle3D_PG2" color="7" fill="1" visible="yes" active="yes"/>
+<layer number="233" name="Eagle3D_PG3" color="7" fill="1" visible="yes" active="yes"/>
 <layer number="248" name="Housing" color="7" fill="1" visible="yes" active="yes"/>
 <layer number="249" name="Edge" color="7" fill="1" visible="yes" active="yes"/>
@@
 <part name="JP10" library="SparkFun-Connectors" deviceset="M09" device="NO_SILK"/>
 <part name="SUPPLY3" library="SparkFun-Aesthetics" deviceset="VCC" device=""/>
-<part name="J1" library="SparkX" deviceset="I2C_STANDARD" device="JS-1MM"/>
-<part name="J2" library="SparkX" deviceset="I2C_STANDARD" device="JS-1MM"/>
-<part name="J3" library="SparkX" deviceset="I2C_STANDARD" device="JS-1MM"/>
+<part name="J1" library="SparkFun-Connectors" deviceset="QWIIC_CONNECTOR" device="JS-1MM"/>
+<part name="J2" library="SparkFun-Connectors" deviceset="QWIIC_CONNECTOR" device="JS-1MM"/>
+<part name="J3" library="SparkFun-Connectors" deviceset="QWIIC_CONNECTOR" device="JS-1MM"/>
 <part name="J4" library="SparkX" deviceset="I2C_STANDARD" device="JS-1MM"/>
 <part name="H1" library="SparkFun-Hardware" deviceset="STAND-OFF" device=""/>
@@
 <part name="SUPPLY7" library="SparkFun-Aesthetics" deviceset="VCC" device=""/>
 <part name="LOGO1" library="SparkFun-Aesthetics" deviceset="OSHW-LOGO" device="M"/>
-<part name="U$4" library="SparkX" deviceset="SPARKX-LOGO" device="5"/>
+<part name="U$4" library="SparkFun-Aesthetics" deviceset="SFE_LOGO_NAME" device=".1_INCH"/>
+<part name="FD1" library="SparkFun-Aesthetics" deviceset="FIDUCIAL" device="UFIDUCIAL"/>
+<part name="FD2" library="SparkFun-Aesthetics" deviceset="FIDUCIAL" device="UFIDUCIAL"/>
+<part name="FD3" library="SparkFun-Aesthetics" deviceset="FIDUCIAL" device="UFIDUCIAL"/>
+<part name="FD4" library="SparkFun-Aesthetics" deviceset="FIDUCIAL" device="UFIDUCIAL"/>
+<part name="LOGO2" library="SparkFun-Aesthetics" deviceset="REVISION" device=""/>
 </parts>
 <sheets>
@@
 <text x="182.88" y="175.26" size="1.778" layer="97" font="vector">VCC Range: 1.9v-3.6v</text>
 <text x="170.688" y="11.43" size="2.54" layer="94">Joel Bartlett</text>
+<text x="174.752" y="7.366" size="2.54" layer="94" font="vector">Andy England</text>
+<text x="236.22" y="7.62" size="2.54" layer="94" font="vector">v01</text>
 </plain>
 <instances>
@@
 <instance part="JP10" gate="G$1" x="226.06" y="91.44"/>
 <instance part="SUPPLY3" gate="G$1" x="93.98" y="129.54"/>
-<instance part="J1" gate="G$1" x="33.02" y="55.88"/>
-<instance part="J2" gate="G$1" x="63.5" y="55.88"/>
-<instance part="J3" gate="G$1" x="91.44" y="55.88"/>
+<instance part="J1" gate="J1" x="33.02" y="55.88"/>
+<instance part="J2" gate="J1" x="63.5" y="55.88"/>
+<instance part="J3" gate="J1" x="91.44" y="55.88"/>
 <instance part="J4" gate="G$1" x="119.38" y="55.88"/>
 <instance part="H1" gate="G$1" x="154.94" y="40.64"/>
@@
 <instance part="SUPPLY7" gate="G$1" x="45.72" y="68.58"/>
 <instance part="LOGO1" gate="G$1" x="236.22" y="45.72"/>
-<instance part="U$4" gate="G$1" x="210.82" y="40.64"/>
+<instance part="U$4" gate="G$1" x="170.18" y="38.1"/>
+<instance part="FD1" gate="G$1" x="154.94" y="38.1"/>
+<instance part="FD2" gate="G$1" x="160.02" y="38.1"/>
+<instance part="FD3" gate="G$1" x="165.1" y="38.1"/>
+<instance part="FD4" gate="G$1" x="170.18" y="38.1"/>
+<instance part="LOGO2" gate="G$1" x="148.59" y="7.366"/>
 </instances>
 <busses>
@@
 <wire x1="104.14" y1="53.34" x2="104.14" y2="48.26" width="0.1524" layer="91"/>
 <pinref part="GND6" gate="1" pin="GND"/>
-<pinref part="J3" gate="G$1" pin="GND"/>
+<pinref part="J3" gate="J1" pin="GND"/>
 </segment>
 <segment>
@@
 <wire x1="76.2" y1="53.34" x2="76.2" y2="48.26" width="0.1524" layer="91"/>
 <pinref part="GND7" gate="1" pin="GND"/>
-<pinref part="J2" gate="G$1" pin="GND"/>
+<pinref part="J2" gate="J1" pin="GND"/>
 </segment>
 <segment>
@@
 <wire x1="45.72" y1="53.34" x2="45.72" y2="48.26" width="0.1524" layer="91"/>
 <pinref part="GND8" gate="1" pin="GND"/>
-<pinref part="J1" gate="G$1" pin="GND"/>
+<pinref part="J1" gate="J1" pin="GND"/>
 </segment>
 </net>
@@
 <wire x1="99.06" y1="60.96" x2="106.68" y2="60.96" width="0.1524" layer="91"/>
 <label x="106.68" y="60.96" size="1.27" layer="95" xref="yes"/>
-<pinref part="J3" gate="G$1" pin="SCL"/>
+<pinref part="J3" gate="J1" pin="SCL"/>
 </segment>
 <segment>
 <wire x1="71.12" y1="60.96" x2="78.74" y2="60.96" width="0.1524" layer="91"/>
 <label x="78.74" y="60.96" size="1.27" layer="95" xref="yes"/>
-<pinref part="J2" gate="G$1" pin="SCL"/>
+<pinref part="J2" gate="J1" pin="SCL"/>
 </segment>
 <segment>
 <wire x1="40.64" y1="60.96" x2="48.26" y2="60.96" width="0.1524" layer="91"/>
 <label x="48.26" y="60.96" size="1.27" layer="95" xref="yes"/>
-<pinref part="J1" gate="G$1" pin="SCL"/>
+<pinref part="J1" gate="J1" pin="SCL"/>
 </segment>
 </net>
@@
 <wire x1="99.06" y1="58.42" x2="106.68" y2="58.42" width="0.1524" layer="91"/>
 <label x="106.68" y="58.42" size="1.27" layer="95" xref="yes"/>
-<pinref part="J3" gate="G$1" pin="SDA"/>
+<pinref part="J3" gate="J1" pin="SDA"/>
 </segment>
 <segment>
 <wire x1="71.12" y1="58.42" x2="78.74" y2="58.42" width="0.1524" layer="91"/>
 <label x="78.74" y="58.42" size="1.27" layer="95" xref="yes"/>
-<pinref part="J2" gate="G$1" pin="SDA"/>
+<pinref part="J2" gate="J1" pin="SDA"/>
 </segment>
 <segment>
 <wire x1="40.64" y1="58.42" x2="48.26" y2="58.42" width="0.1524" layer="91"/>
 <label x="48.26" y="58.42" size="1.27" layer="95" xref="yes"/>
-<pinref part="J1" gate="G$1" pin="SDA"/>
+<pinref part="J1" gate="J1" pin="SDA"/>
 </segment>
 </net>
@@
 <wire x1="104.14" y1="55.88" x2="104.14" y2="68.58" width="0.1524" layer="91"/>
 <pinref part="SUPPLY5" gate="G$1" pin="VCC"/>
-<pinref part="J3" gate="G$1" pin="VCC"/>
+<pinref part="J3" gate="J1" pin="VCC"/>
 </segment>
 <segment>
@@
 <wire x1="76.2" y1="55.88" x2="76.2" y2="68.58" width="0.1524" layer="91"/>
 <pinref part="SUPPLY6" gate="G$1" pin="VCC"/>
-<pinref part="J2" gate="G$1" pin="VCC"/>
+<pinref part="J2" gate="J1" pin="VCC"/>
 </segment>
 <segment>
@@
 <wire x1="45.72" y1="55.88" x2="45.72" y2="68.58" width="0.1524" layer="91"/>
 <pinref part="SUPPLY7" gate="G$1" pin="VCC"/>
-<pinref part="J1" gate="G$1" pin="VCC"/>
-</segment>
-</net>
+<pinref part="J1" gate="J1" pin="VCC"/>
+</segment>
+</net>

Commit message: updated version silk, added gnd stitching
Other:
- note added: "v10"
- note removed: "v01"
Changed lines of the file:
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@@
 <text x="170.688" y="11.43" size="2.54" layer="94">Joel Bartlett</text>
 <text x="174.752" y="7.366" size="2.54" layer="94" font="vector">Andy England</text>
-<text x="236.22" y="7.62" size="2.54" layer="94" font="vector">v01</text>
+<text x="236.22" y="7.62" size="2.54" layer="94" font="vector">v10</text>
 </plain>
 <instances>
